File: SOURCES/KiCAD/USBi_Programmer.kicad_pcb (KiCad board)
At the start: 2 copper layers, 40 x 40 mm, 24 parts, among them P1 CONN_02X10, P2 CONN_02X05, P3 CONN_01X02, P4 CONN_02X10, Q1 Q_NMOS_DGS, Q2 Q_NMOS_DGS

Commit message: V0.2: Move holes & disconnect 2 pins from pinheader
These pins usually had to be cut out from the main cypress board.
Now that they're disconnected, there's no need anymore to cut them.

Also the mounting holes didn't fit exactly to the holes on the cypress main board.
Parts:
- moved REF** 0.50 mm to (137.0, 175.8)
- moved REF** 0.50 mm to (103.0, 175.8)
Connections:
- P1 pad 10: GND -> Net-(P1-Pad10)
- P1 pad 19: +3V3 -> Net-(P1-Pad19)
Routing:
- net +3V3: track 39.7 -> 36.6 mm
- net GND: track 133.2 -> 134.2 mm
- net Net-(P1-Pad15): track 34.2 -> 34.8 mm
Other:
- board text added: "freeUSBi v0.2"
- board text removed: "freeUSBi v0.1"
